File: ECAD/DIC/untitled.kicad_sch (KiCad schematic)
At the start: 41 parts, among them Q2 BC846, Q3 BC846, Q4 BC846, Q5 BC846, Q6 BC846, Q8 BC846, U10 ADA4500-2, U9 ADA4500-2

Commit message: few small changes
Parts:
- added R58, R59, R60: 10kR 0603, Resistor_SMD:R_0603_1608Metric_Pad0.98x0.95mm_HandSolder, symbol Device:R
Connections:
- net +3.3V: now also R58.1, R59.1, R60.1
- net ADC1_CTRL: now also R58.2
- net ADC2_CTRL: now also R60.2
- net ADC3_CTRL: now also R59.2
Changed lines of the file:
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@@
   (junction (at 86.36 128.27) (diameter 0) (color 0 0 0 0)
   )
+  (junction (at 77.47 168.91) (diameter 0) (color 0 0 0 0)
+  )
   (junction (at 82.55 128.27) (diameter 0) (color 0 0 0 0)
   )
@@
   (junction (at 111.76 72.39) (diameter 0) (color 0 0 0 0)
   )
+  (junction (at 72.39 83.82) (diameter 0) (color 0 0 0 0)
+  )
+  (junction (at 182.88 80.01) (diameter 0) (color 0 0 0 0)
+  )
   (junction (at 111.76 33.02) (diameter 0) (color 0 0 0 0)
   )
@@
     (stroke (width 0) (type default))
   )
+  (wire (pts (xy 72.39 171.45) (xy 72.39 168.91))
+    (stroke (width 0) (type default))
+  )
   (wire (pts (xy 81.28 72.39) (xy 91.44 72.39))
     (stroke (width 0) (type default))
@@
     (stroke (width 0) (type default))
   )
+  (wire (pts (xy 77.47 168.91) (xy 77.47 167.64))
+    (stroke (width 0) (type default))
+  )
   (wire (pts (xy 96.52 157.48) (xy 96.52 158.75))
     (stroke (width 0) (type default))
@@
     (stroke (width 0) (type default))
   )
+  (wire (pts (xy 72.39 168.91) (xy 77.47 168.91))
+    (stroke (width 0) (type default))
+  )
   (wire (pts (xy 96.52 128.27) (xy 100.33 128.27))
     (stroke (width 0) (type default))
@@
     (stroke (width 0) (type default))
   )
+  (wire (pts (xy 67.31 86.36) (xy 67.31 83.82))
+    (stroke (width 0) (type default))
+  )
   (wire (pts (xy 222.25 40.64) (xy 222.25 41.91))
     (stroke (width 0) (type default))
@@
     (stroke (width 0) (type default))
   )
+  (wire (pts (xy 72.39 83.82) (xy 72.39 82.55))
+    (stroke (width 0) (type default))
+  )
   (wire (pts (xy 60.96 170.18) (xy 60.96 167.64))
     (stroke (width 0) (type default))
@@
     (stroke (width 0) (type default))
   )
+  (wire (pts (xy 177.8 80.01) (xy 182.88 80.01))
+    (stroke (width 0) (type default))
+  )
   (wire (pts (xy 86.36 157.48) (xy 96.52 157.48))
     (stroke (width 0) (type default))
@@
     (stroke (width 0) (type default))
   )
+  (wire (pts (xy 67.31 83.82) (xy 72.39 83.82))
+    (stroke (width 0) (type default))
+  )
   (wire (pts (xy 73.66 43.18) (xy 77.47 43.18))
     (stroke (width 0) (type default))
@@
     (stroke (width 0) (type default))
   )
-  (wire (pts (xy 77.47 170.18) (xy 77.47 167.64))
+  (wire (pts (xy 77.47 170.18) (xy 77.47 168.91))
     (stroke (width 0) (type default))
   )
@@
     (stroke (width 0) (type default))
   )
-  (wire (pts (xy 72.39 85.09) (xy 72.39 82.55))
+  (wire (pts (xy 72.39 85.09) (xy 72.39 83.82))
     (stroke (width 0) (type default))
   )
@@
     (stroke (width 0) (type default))
   )
-  (wire (pts (xy 182.88 81.28) (xy 182.88 78.74))
+  (wire (pts (xy 182.88 81.28) (xy 182.88 80.01))
     (stroke (width 0) (type default))
   )
@@
   )
   (wire (pts (xy 115.57 130.81) (xy 116.84 130.81))
+    (stroke (width 0) (type default))
+  )
+  (wire (pts (xy 177.8 82.55) (xy 177.8 80.01))
+    (stroke (width 0) (type default))
+  )
+  (wire (pts (xy 182.88 80.01) (xy 182.88 78.74))
     (stroke (width 0) (type default))
   )
@@
     )
   )
+  (symbol (lib_id "power:+3.3V") (at 72.39 179.07 180) (unit 1)
+    (in_bom yes) (on_board yes) (dnp no) (fields_autoplaced)
+    (property "Reference" "#PWR067" (at 72.39 175.26 0)
+      (effects (font (size 1.27 1.27)) hide)
+    )
+    (property "Value" "+3.3V" (at 72.39 184.15 0)
+      (effects (font (size 1.27 1.27)))
+    )
+    (property "Footprint" "" (at 72.39 179.07 0)
+      (effects (font (size 1.27 1.27)) hide)
+    )
+    (property "Datasheet" "" (at 72.39 179.07 0)
+      (effects (font (size 1.27 1.27)) hide)
+    )
+    (pin "1")
+    (instances
+      (project "DIC"
+        (path "/64369a6c-13db-47f8-8de7-12b4f0b9bc27/686c77eb-8dbe-46c8-ba78-2cfcedb8436d"
+          (reference "#PWR067") (unit 1)
+        )
+      )
+    )
+  )
   (symbol (lib_id "Device:R") (at 69.85 43.18 90) (unit 1)
     (in_bom yes) (on_board yes) (dnp no)
@@
         (path "/64369a6c-13db-47f8-8de7-12b4f0b9bc27/686c77eb-8dbe-46c8-ba78-2cfcedb8436d"
           (reference "R44") (unit 1)
+        )
+      )
+    )
+  )
+  (symbol (lib_id "power:+3.3V") (at 177.8 90.17 180) (unit 1)
+    (in_bom yes) (on_board yes) (dnp no) (fields_autoplaced)
+    (property "Reference" "#PWR068" (at 177.8 86.36 0)
+      (effects (font (size 1.27 1.27)) hide)
+    )
+    (property "Value" "+3.3V" (at 177.8 95.25 0)
+      (effects (font (size 1.27 1.27)))
+    )
+    (property "Footprint" "" (at 177.8 90.17 0)
+      (effects (font (size 1.27 1.27)) hide)
+    )
+    (property "Datasheet" "" (at 177.8 90.17 0)
+      (effects (font (size 1.27 1.27)) hide)
+    )
+    (pin "1")
+    (instances
+      (project "DIC"
+        (path "/64369a6c-13db-47f8-8de7-12b4f0b9bc27/686c77eb-8dbe-46c8-ba78-2cfcedb8436d"
+          (reference "#PWR068") (unit 1)
+        )
+      )
+    )
+  )
+  (symbol (lib_id "Device:R") (at 177.8 86.36 180) (unit 1)
+    (in_bom yes) (on_board yes) (dnp no)
+    (property "Reference" "R60" (at 177.8 86.36 90)
+      (effects (font (size 1.27 1.27)))
+    )
+    (property "Value" "10kR 0603" (at 175.26 86.36 90)
+      (effects (font (size 1.27 1.27)))
+    )
+    (property "Footprint" "Resistor_SMD:R_0603_1608Metric_Pad0.98x0.95mm_HandSolder" (at 179.578 86.36 90)
+      (effects (font (size 1.27 1.27)) hide)
+    )
+    (property "Datasheet" "~" (at 177.8 86.36 0)
+      (effects (font (size 1.27 1.27)) hide)
+    )
+    (pin "1")
+    (pin "2")
+    (instances
+      (project "DIC"
+        (path "/64369a6c-13db-47f8-8de7-12b4f0b9bc27/686c77eb-8dbe-46c8-ba78-2cfcedb8436d"
+          (reference "R60") (unit 1)
         )
       )
@@
     )
   )
+  (symbol (lib_id "Device:R") (at 67.31 90.17 180) (unit 1)
+    (in_bom yes) (on_board yes) (dnp no)
+    (property "Reference" "R58" (at 67.31 90.17 90)
+      (effects (font (size 1.27 1.27)))
+    )
+    (property "Value" "10kR 0603" (at 64.77 90.17 90)
+      (effects (font (size 1.27 1.27)))
+    )
+    (property "Footprint" "Resistor_SMD:R_0603_1608Metric_Pad0.98x0.95mm_HandSolder" (at 69.088 90.17 90)
+      (effects (font (size 1.27 1.27)) hide)
+    )
+    (property "Datasheet" "~" (at 67.31 90.17 0)
+      (effects (font (size 1.27 1.27)) hide)
+    )
+    (pin "1")
+    (pin "2")
+    (instances
+      (project "DIC"
+        (path "/64369a6c-13db-47f8-8de7-12b4f0b9bc27/686c77eb-8dbe-46c8-ba78-2cfcedb8436d"
+          (reference "R58") (unit 1)
+        )
+      )
+    )
+  )
   (symbol (lib_id "Device:R") (at 180.34 39.37 90) (unit 1)
     (in_bom yes) (on_board yes) (dnp no)
@@
         (path "/64369a6c-13db-47f8-8de7-12b4f0b9bc27/686c77eb-8dbe-46c8-ba78-2cfcedb8436d"
           (reference "R30") (unit 1)
+        )
+      )
+    )
+  )
+  (symbol (lib_id "Device:R") (at 72.39 175.26 180) (unit 1)
+    (in_bom yes) (on_board yes) (dnp no)
+    (property "Reference" "R59" (at 72.39 175.26 90)
+      (effects (font (size 1.27 1.27)))
+    )
+    (property "Value" "10kR 0603" (at 69.85 175.26 90)
+      (effects (font (size 1.27 1.27)))
+    )
+    (property "Footprint" "Resistor_SMD:R_0603_1608Metric_Pad0.98x0.95mm_HandSolder" (at 74.168 175.26 90)
+      (effects (font (size 1.27 1.27)) hide)
+    )
+    (property "Datasheet" "~" (at 72.39 175.26 0)
+      (effects (font (size 1.27 1.27)) hide)
+    )
+    (pin "1")
+    (pin "2")
+    (instances
+      (project "DIC"
+        (path "/64369a6c-13db-47f8-8de7-12b4f0b9bc27/686c77eb-8dbe-46c8-ba78-2cfcedb8436d"
+          (reference "R59") (unit 1)
         )
       )
@@
         )
       )
+    )
+  )
+  (symbol (lib_id "power:+3.3V") (at 67.31 93.98 180) (unit 1)
+    (in_bom yes) (on_board yes) (dnp no) (fields_autoplaced)
+    (property "Reference" "#PWR066" (at 67.31 90.17 0)
+      (effects (font (size 1.27 1.27)) hide)
+    )
+    (property "Value" "+3.3V" (at 67.31 99.06 0)
+      (effects (font (size 1.27 1.27)))
+    )
+    (property "Footprint" "" (at 67.31 93.98 0)
+      (effects (font (size 1.27 1.27)) hide)
+    )
+    (property "Datasheet" "" (at 67.31 93.98 0)
+      (effects (font (size 1.27 1.27)) hide)
+    )
+    (pin "1")
+    (instances
+      (project "DIC"
+        (path "/64369a6c-13db-47f8-8de7-12b4f0b9bc27/686c77eb-8dbe-46c8-ba78-2cfcedb8436d"
+          (reference "#PWR066") (unit 1)
+        )
+      )
