File: ECAD/DIC/DIC.kicad_pcb (KiCad board)
At the start: 2 copper layers, 68.1 x 55.2 mm, 69 parts, among them J1 Solder Pad, J10 Solder Pad, J11 Solder Pad, J12 Solder Pad, J13 Solder Pad, J14 Solder Pad, J15 Solder Pad, J16 Solder Pad, J17 Solder Pad, J18 Conn_01x06_Socket, J19 Conn_01x06_Socket, J2 Solder Pad, J20 Conn_01x06_Socket, J22 Conn_01x06_Socket, J3 Solder Pad, J4 Solder Pad, J5 Solder Pad, J6 Solder Pad, J7 Solder Pad, J8 Solder Pad, J9 Solder Pad, U1 R-78E5.0-1.0, U2 MCP130-270, U3 STM32F072RBTx, U5 R-78E3.3-1.0, U7 MCP2562-E-SN, Y1 LFXTAL051370

Commit message: switch to ribbon cable pcb interconnect
Parts:
- removed CAN1: Micro-Fit_3.0_43045-0412, Lukas:Molex_Micro-Fit_3.0_43045-0412_2x02_P3.00mm_Vertical
- removed J10, J11, J12, J13, J14, J15, J16, J17, J2, J3, J4, J5, J6, J7, J8, J9: Solder Pad, Jumper:SolderJumper-2_P1.3mm_Bridged2Bar_RoundedPad1.0x1.5mm
- removed J18, J19, J20, J22: Conn_01x06_Socket, Connector_PinSocket_2.54mm:PinSocket_1x06_P2.54mm_Vertical
- removed TP1, TP2: TestPoint D1mm_Pad, TestPoint:TestPoint_Pad_D1.0mm
- added 12VGood1: LED Green, LED_SMD:LED_0805_2012Metric_Pad1.15x1.40mm_HandSolder, B.Cu at (28.2, 50.5)
- added C22: 10uF 0805 16V, Capacitor_SMD:C_0805_2012Metric_Pad1.18x1.45mm_HandSolder, B.Cu at (14.6, 61.1)
- added C23: 10uF 0805 16V, Capacitor_SMD:C_0805_2012Metric_Pad1.18x1.45mm_HandSolder, B.Cu at (23.1, 48.9)
- added C24: 160nF 0603 6.3V, Capacitor_SMD:C_0603_1608Metric_Pad1.08x0.95mm_HandSolder, B.Cu at (50.3, 32.9)
- added C25: 160nF 0603 6.3V, Capacitor_SMD:C_0603_1608Metric_Pad1.08x0.95mm_HandSolder, B.Cu at (48.3, 46.1)
- added C26: 10uF 0805 6.3V, Capacitor_SMD:C_0805_2012Metric_Pad1.18x1.45mm_HandSolder, B.Cu at (57.1, 47.2)
- added C27: 10uF 0805 6.3V, Capacitor_SMD:C_0805_2012Metric_Pad1.18x1.45mm_HandSolder, B.Cu at (55.4, 23.4)
- added C28: 160nF 0603 6.3V, Capacitor_SMD:C_0603_1608Metric_Pad1.08x0.95mm_HandSolder, B.Cu at (53.5, 18.3)
- added C29: 160nF 0603 6.3V, Capacitor_SMD:C_0603_1608Metric_Pad1.08x0.95mm_HandSolder, B.Cu at (50.5, 26.0)
- added C30: 100nF 0603 6.3V, Capacitor_SMD:C_0603_1608Metric_Pad1.08x0.95mm_HandSolder, B.Cu at (50.8, 41.4)
- added C31: 100nF 0603 6.3V, Capacitor_SMD:C_0603_1608Metric_Pad1.08x0.95mm_HandSolder, B.Cu at (58.8, 24.6)
- added D1: NSVRB751V40T1G, Diode_SMD:D_SOD-323_HandSoldering, B.Cu at (52.2, 32.5)
- added D10: Z 3.3V, Diode_SMD:D_SOD-323_HandSoldering, B.Cu at (31.4, 61.1)
- added D2: NSVRB751V40T1G, Diode_SMD:D_SOD-323_HandSoldering, B.Cu at (47.4, 48.9)
- added D3: NSVRB751V40T1G, Diode_SMD:D_SOD-323_HandSoldering, B.Cu at (58.7, 22.2)
- added D4: DESD5V0S1BA-7, Diode_SMD:D_SOD-323, B.Cu at (36.6, 19.1)
- added D5: DESD5V0S1BA-7, Diode_SMD:D_SOD-323, B.Cu at (39.2, 18.2)
- added D8: NSVRB751V40T1G, Diode_SMD:D_SOD-323_HandSoldering, B.Cu at (52.3, 24.3)
- added JP1: Jumper_2_Open, Jumper:SolderJumper-2_P1.3mm_Open_RoundedPad1.0x1.5mm, B.Cu at (14.0, 51.1)
- added JP2: Jumper_2_Open, Jumper:SolderJumper-2_P1.3mm_Open_RoundedPad1.0x1.5mm, B.Cu at (20.3, 51.7)
- added Q1: BC846, Package_TO_SOT_SMD:SOT-23, B.Cu at (68.1, 33.3)
- added Q2: BC846, Package_TO_SOT_SMD:SOT-23, B.Cu at (65.8, 38.7)
- added Q3: BC846, Package_TO_SOT_SMD:SOT-23, B.Cu at (59.1, 32.8)
- added Q4: BC846, Package_TO_SOT_SMD:SOT-23, B.Cu at (67.2, 47.6)
- added Q5: BC846, Package_TO_SOT_SMD:SOT-23, B.Cu at (62.9, 49.6)
- added Q6: BC846, Package_TO_SOT_SMD:SOT-23, B.Cu at (67.3, 23.9)
- added Q7: BC846, Package_TO_SOT_SMD:SOT-23, B.Cu at (63.6, 29.8)
- added Q8: BC846, Package_TO_SOT_SMD:SOT-23, B.Cu at (69.8, 17.5)
- added R12: 100 0603, Resistor_SMD:R_0603_1608Metric_Pad0.98x0.95mm_HandSolder, B.Cu at (65.8, 41.4)
- added R13: 100 0603, Resistor_SMD:R_0603_1608Metric_Pad0.98x0.95mm_HandSolder, B.Cu at (64.4, 33.5)
- added R14: 82kR 0603 0.1%, Resistor_SMD:R_0603_1608Metric_Pad0.98x0.95mm_HandSolder, B.Cu at (58.9, 37.6)
- added R15: 2.2MR 0603 0.1%, Resistor_SMD:R_0603_1608Metric_Pad0.98x0.95mm_HandSolder, B.Cu at (57.1, 36.1)
- added R16: 5kR 0603 0.1%, Resistor_SMD:R_0603_1608Metric_Pad0.98x0.95mm_HandSolder, B.Cu at (62.4, 37.6)
- added R17: 5kR 0603 0.1%, Resistor_SMD:R_0603_1608Metric_Pad0.98x0.95mm_HandSolder, B.Cu at (70.7, 31.0)
- added R18: 100 0603, Resistor_SMD:R_0603_1608Metric_Pad0.98x0.95mm_HandSolder, B.Cu at (55.0, 33.7)
- added R19: 39kR 0603 0.1%, Resistor_SMD:R_0603_1608Metric_Pad0.98x0.95mm_HandSolder, B.Cu at (54.5, 37.0)
- added R20: 150kR 0603 0.1%, Resistor_SMD:R_0603_1608Metric_Pad0.98x0.95mm_HandSolder, B.Cu at (57.4, 39.1)
- added R21: 1k 0603 0.1%, Resistor_SMD:R_0603_1608Metric_Pad0.98x0.95mm_HandSolder, B.Cu at (51.3, 37.0)
- added R22: 100 0603 0.1%, Resistor_SMD:R_0603_1608Metric_Pad0.98x0.95mm_HandSolder, B.Cu at (51.2, 35.4)
- added R23: 100 0603, Resistor_SMD:R_0603_1608Metric_Pad0.98x0.95mm_HandSolder, B.Cu at (68.2, 51.3)
- added R24: 82kR 0603 0.1%, Resistor_SMD:R_0603_1608Metric_Pad0.98x0.95mm_HandSolder, B.Cu at (62.4, 43.8)
- added R25: 2.2MR 0603 0.1%, Resistor_SMD:R_0603_1608Metric_Pad0.98x0.95mm_HandSolder, B.Cu at (64.8, 44.7)
- added R26: 2.2MR 0603 0.1%, Resistor_SMD:R_0603_1608Metric_Pad0.98x0.95mm_HandSolder, B.Cu at (67.7, 28.8)
- added R27: 5kR 0603 0.1%, Resistor_SMD:R_0603_1608Metric_Pad0.98x0.95mm_HandSolder, B.Cu at (67.2, 43.8)
- added R28: 100 0603, Resistor_SMD:R_0603_1608Metric_Pad0.98x0.95mm_HandSolder, B.Cu at (59.7, 49.6)
- added R29: 39kR 0603 0.1%, Resistor_SMD:R_0603_1608Metric_Pad0.98x0.95mm_HandSolder, B.Cu at (60.6, 46.2)
- added R30: 150kR 0603 0.1%, Resistor_SMD:R_0603_1608Metric_Pad0.98x0.95mm_HandSolder, B.Cu at (50.8, 42.9)
- added R31: 100 0603, Resistor_SMD:R_0603_1608Metric_Pad0.98x0.95mm_HandSolder, B.Cu at (59.3, 28.7)
- added R32: 1k 0603 0.1%, Resistor_SMD:R_0603_1608Metric_Pad0.98x0.95mm_HandSolder, B.Cu at (51.8, 45.7)
- added R33: 100 0603 0.1%, Resistor_SMD:R_0603_1608Metric_Pad0.98x0.95mm_HandSolder, B.Cu at (49.1, 44.6)
- added R34: 1k 0603 0.1%, Resistor_SMD:R_0603_1608Metric_Pad0.98x0.95mm_HandSolder, B.Cu at (53.8, 27.7)
- added R35: 100 0603, Resistor_SMD:R_0603_1608Metric_Pad0.98x0.95mm_HandSolder, B.Cu at (67.1, 26.4)
- added R36: 100 0603 0.1%, Resistor_SMD:R_0603_1608Metric_Pad0.98x0.95mm_HandSolder, B.Cu at (53.8, 26.0)
- added R37: 82kR 0603 0.1%, Resistor_SMD:R_0603_1608Metric_Pad0.98x0.95mm_HandSolder, B.Cu at (71.0, 23.2)
- added R38: 82kR 0603 0.1%, Resistor_SMD:R_0603_1608Metric_Pad0.98x0.95mm_HandSolder, B.Cu at (70.7, 27.7)
- added R39: 39kR 0603 0.1%, Resistor_SMD:R_0603_1608Metric_Pad0.98x0.95mm_HandSolder, B.Cu at (69.2, 29.8)
- added R40: 150kR 0603 0.1%, Resistor_SMD:R_0603_1608Metric_Pad0.98x0.95mm_HandSolder, B.Cu at (62.9, 27.2)
- added R41: 2.2MR 0603 0.1%, Resistor_SMD:R_0603_1608Metric_Pad0.98x0.95mm_HandSolder, B.Cu at (59.4, 18.8)
- added R42: 5kR 0603 0.1%, Resistor_SMD:R_0603_1608Metric_Pad0.98x0.95mm_HandSolder, B.Cu at (71.0, 25.1)
- added R43: 100 0603, Resistor_SMD:R_0603_1608Metric_Pad0.98x0.95mm_HandSolder, B.Cu at (65.8, 17.9)
- added R44: 39kR 0603 0.1%, Resistor_SMD:R_0603_1608Metric_Pad0.98x0.95mm_HandSolder, B.Cu at (71.0, 21.6)
- added R45: 150kR 0603 0.1%, Resistor_SMD:R_0603_1608Metric_Pad0.98x0.95mm_HandSolder, B.Cu at (69.5, 20.1)
- added R46: 1k 0603 0.1%, Resistor_SMD:R_0603_1608Metric_Pad0.98x0.95mm_HandSolder, B.Cu at (55.9, 18.9)
- added R47: 100 0603 0.1%, Resistor_SMD:R_0603_1608Metric_Pad0.98x0.95mm_HandSolder, B.Cu at (55.9, 17.4)
- added U10: ADA4500-2, Package_SO:MSOP-8_3x3mm_P0.65mm, B.Cu at (63.5, 23.2)
- added U8: NCP1117-12, Package_TO_SOT_SMD:TO-252-2, B.Cu at (18.9, 56.5)
- added U9: ADA4500-2, Package_SO:MSOP-8_3x3mm_P0.65mm, B.Cu at (57.0, 41.9)
- J1: value Solder Pad -> WE 62702621621; footprint Jumper:SolderJumper-2_P1.3mm_Bridged2Bar_RoundedPad1.0x1.5mm -> Connector_PinHeader_1.27mm:PinHeader_2x17_P1.27mm_Vertical
- JTAG1: footprint Connector_PinHeader_1.27mm:PinHeader_2x05_P1.27mm_Vertical -> Connector_PinHeader_1.27mm:PinHeader_2x07_P1.27mm_Vertical
- R4: value 470R 0603 -> 1kR 0603
- R5, R7: value 1kR 0603 -> ? 0603
- R6: value 330R 0603 -> 1kR 0603
- Y1: value LFXTAL051370 -> WE830055951; footprint Crystal:Crystal_SMD_HC49-SD_HandSoldering -> Oscillator:Oscillator_SMD_EuroQuartz_XO32-4Pin_3.2x2.5mm_HandSoldering
- moved JTAG1 64.1 mm to (76.8, 14.5)
- moved R5 30.2 mm to (17.7, 49.7)
- moved J1 30.1 mm to (16.5, 23.6), turned to 180 degrees
- moved R8 26.8 mm to (25.5, 50.2), turned to -90 degrees
- moved R7 26.5 mm to (20.3, 48.4), turned to -90 degrees
- moved C17 16.7 mm to (39.9, 22.0)
- moved C18 16.7 mm to (39.9, 20.2)
- moved R10 16.7 mm to (48.1, 19.6)
- moved U7 16.7 mm to (44.5, 21.2)
- moved R11 15.1 mm to (44.5, 16.7)
- moved C5 4.38 mm to (34.4, 44.5), turned to 90 degrees
- moved C14 3.32 mm to (42.4, 49.9)
- moved C10 2.78 mm to (41.5, 41.1), turned to -90 degrees
- moved C15 2.34 mm to (45.3, 49.0), turned to 90 degrees
- moved C9 1.48 mm to (43.1, 40.1), turned to -90 degrees
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Connections:
- net /Display_nCS renamed /nCS_Display
- net /D/nC renamed /D_nC_Display
- net /SPI1_CLK renamed /SPI1_SCK_Display
- net /SPI1_MOSI renamed /SPI1_MOSI_Display
- C19 pad 2: +BATT -> +12V
- J1 pad 1: Net-(J1-Pin_1) -> Analog1_In
- J1 pad 2: (no net) -> Analog0_In
- JTAG1 pad 1: +3.3V -> unconnected-(JTAG1-Pin_1-Pad1)
- JTAG1 pad 10: JTMS/SWDIO -> JTDI/NC
- JTAG1 pad 2: GND -> unconnected-(JTAG1-Pin_2-Pad2)
- JTAG1 pad 3: GND -> +3.3V
- JTAG1 pad 4: JRCLK -> JTMS/SWDIO
- JTAG1 pad 6: NRST -> JCLK/SWCLK
- JTAG1 pad 7: JTDI/NC -> GND
- JTAG1 pad 9: JCLK/SWCLK -> unconnected-(JTAG1-Pin_9-Pad9)
- R11 pad 1: CAN1_L -> CAN1_N
- R11 pad 2: CAN1_H -> CAN1_P
- R5 pad 1: !RTS -> GND
- R5 pad 2: Net-(U3-PB3) -> Net-(JP1-B)
- R7 pad 1: Net-(U3-PA9) -> Net-(JP1-B)
- R7 pad 2: USART1_RX -> +12V
- R8 pad 1: USART1_TX -> Net-(12VGood1-A)
- R8 pad 2: Net-(U3-PA10) -> +12V
- U3 pad 10: Net-(J1-Pin_1) -> unconnected-(U3-PC2-Pad10)
- U3 pad 11: Net-(J2-Pin_1) -> /SPI2_MOSI_RGBLED
- U3 pad 14: Net-(J7-Pin_1) -> ADC0
- U3 pad 15: Net-(J8-Pin_1) -> ADC1
- U3 pad 16: Net-(J9-Pin_1) -> ADC2
- U3 pad 17: Net-(J17-Pin_1) -> ADC3
- U3 pad 2: GPO2_CTRL -> unconnected-(U3-PC13-Pad2)
- U3 pad 24: Net-(J3-Pin_1) -> /nRES_Display
- U3 pad 25: Net-(J4-Pin_1) -> unconnected-(U3-PC5-Pad25)
- U3 pad 26: RX_IND -> ADC2_NTC_CTRL
- U3 pad 27: TX_IND -> ADC1_NTC_CTRL
- U3 pad 28: Radio_RESET -> ADC0_NTC_CTRL
- U3 pad 29: Net-(J11-Pin_1) -> /SPI2_SCK_RGBLED
- U3 pad 3: GPO3_CTRL -> unconnected-(U3-PC14-Pad3)
- U3 pad 30: Net-(J12-Pin_1) -> ADC1_CTRL
- U3 pad 33: Net-(J13-Pin_1) -> ADC2_CTRL
- U3 pad 34: Net-(J14-Pin_1) -> ADC3_CTRL
- U3 pad 35: Net-(J15-Pin_1) -> GPIO3_In
- U3 pad 36: Net-(J16-Pin_1) -> GPIO3_5VOut
- U3 pad 37: Net-(J5-Pin_1) -> GPIO3_12VOut
- U3 pad 38: Net-(J6-Pin_1) -> GPIO2_In
- U3 pad 39: GPI1_CTRL -> GPIO2_5VOut
- U3 pad 4: GPO4_CTRL -> unconnected-(U3-PC15-Pad4)
- U3 pad 40: GPI2_CTRL -> GPIO2_12VOut
- U3 pad 41: /nRES -> GPIO1_In
- U3 pad 42: Net-(U3-PA9) -> GPIO1_5VOut
- U3 pad 43: Net-(U3-PA10) -> GPIO1_12VOut
- U3 pad 51: GPI3_CTRL -> GPIO6_In
- U3 pad 52: GPI4_CTRL -> GPIO6_5VOut
- U3 pad 53: GPO1_CTRL -> GPIO6_12VOut
- U3 pad 54: unconnected-(U3-PD2-Pad54) -> GPIO5_In
- U3 pad 55: Net-(U3-PB3) -> GPIO5_5VOut
- U3 pad 56: Wake-Up -> GPIO5_12VOut
- U3 pad 57: Mode_1 -> GPIO4_In
- U3 pad 58: /I2C_CLK -> GPIO4_5VOut
- U3 pad 59: /I2C_Data -> GPIO4_12VOut
- U3 pad 61: Radio_BOOT -> ADC3_NTC_CTRL
- U3 pad 62: Net-(J10-Pin_1) -> ADC0_CTRL
- U4 pad 1: /I2C_Data -> /SPI2_MOSI_RGBLED
- U4 pad 2: /I2C_CLK -> /SPI2_SCK_RGBLED
- U6 pad 21: +BATT -> +12V
- U6 pad 22: +BATT -> +12V
- U6 pad 30: /nRES -> /nRES_Display
- U6 pad 39: +BATT -> +12V
- U6 pad 40: +BATT -> +12V
- U7 pad 6: CAN1_L -> CAN1_N
- U7 pad 7: CAN1_H -> CAN1_P
- Y1 pad 2: Net-(U3-PF0) -> GND
Routing:
- net +3.3V: track 258.6 -> 111.5 mm, vias 10 -> 18
- net +12V: track 0.00 -> 110.9 mm, vias 0 -> 6
- net Analog2_In: track 0.00 -> 99.9 mm, vias 0 -> 1
- net GPIO3_5VOut: track 0.00 -> 92.1 mm, vias 0 -> 4
- net GND: track 64.8 -> 146.7 mm, vias 59 -> 42
- net GPIO2_In: track 0.00 -> 80.6 mm, vias 0 -> 2
- net Analog1_In: track 0.00 -> 80.4 mm, vias 0 -> 1
- net GPIO2_12VOut: track 0.00 -> 79.2 mm, vias 0 -> 2
- net Analog0_In: track 0.00 -> 71.8 mm, vias 0 -> 1
- net GPIO1_5VOut: track 0.00 -> 66.7 mm, vias 0 -> 2
- net Analog3_In: track 0.00 -> 65.1 mm, vias 0 -> 2
- net GPO2_CTRL: track 63.2 -> 0.00 mm, vias 4 -> 0
- net ADC2_NTC_CTRL: track 0.00 -> 61.9 mm, vias 0 -> 2
- net GPIO3_In: track 0.00 -> 60.4 mm, vias 0 -> 3
- net Reset: track 15.0 -> 74.7 mm, vias 4 -> 3
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- added copper zone on In2.Cu, net +3.3V
- added copper zone on In1.Cu, net GND
- removed copper zone on B.Cu, net GND
- removed copper zone on F.Cu, net GND
Other:
- copper layers 2 -> 4

Commit message: finisjed PCB projekt
Parts:
- removed J1: WE 62702621621, Connector_PinHeader_1.27mm:PinHeader_2x17_P1.27mm_Vertical
- added J2: Conn_02x05_Top_Bottom, Connector_PinHeader_1.27mm:PinHeader_2x05_P1.27mm_Vertical, B.Cu at (76.2, 14.9)
- added J3: Conn_02x05_Top_Bottom, Connector_PinHeader_1.27mm:PinHeader_2x05_P1.27mm_Vertical, B.Cu at (75.8, 54.5)
- added J4: Conn_02x05_Top_Bottom, Connector_PinHeader_1.27mm:PinHeader_2x05_P1.27mm_Vertical, B.Cu at (16.1, 20.7)
- added J5: Conn_02x05_Top_Bottom, Connector_PinHeader_1.27mm:PinHeader_2x05_P1.27mm_Vertical, B.Cu at (16.9, 54.5)
- moved JP1 63.9 mm to (77.9, 50.3)
- moved R5 59.7 mm to (77.3, 47.0), turned to -90 degrees
- moved R7 58.0 mm to (78.1, 43.7), turned to 90 degrees
- moved C22 55.7 mm to (70.0, 54.6), turned to 180 degrees
- moved U8 55.1 mm to (73.0, 46.5), turned to 90 degrees
- moved JP2 50.1 mm to (70.1, 57.4), turned to 0 degrees
- moved C23 47.9 mm to (70.2, 40.4), turned to 180 degrees
- moved R8 45.6 mm to (69.6, 38.4), turned to 0 degrees
- moved 12VGood 43.7 mm to (69.5, 36.2)
- moved D4 17.7 mm to (53.8, 15.2), turned to 0 degrees
- moved JTAG1 15.2 mm to (76.8, 29.7)
- moved D5 10.8 mm to (49.9, 19.6), turned to -90 degrees
- renumbered 12VGood1 to 12VGood, 3V3Good1 to 3V3Good, 5VGood1 to 5VGood, Error1 to Error, Heart1 to Heart
Routing:
- net Analog2_In: track 99.9 -> 32.9 mm, vias 1 -> 0
- net Analog3_In: track 65.1 -> 7.65 mm, vias 2 -> 1
- net +BATT: track 118.5 -> 61.7 mm, vias 5 -> 2
- net Analog0_In: track 71.8 -> 18.9 mm, vias 1 -> 2
- net Analog1_In: track 80.4 -> 30.3 mm, vias 1 -> 0
- net +3.3V: track 111.5 -> 63.7 mm, vias 18 -> 13
- net +5V: track 149.4 -> 191.0 mm, vias 8 -> 6
- net GPIO3_5VOut: track 92.1 -> 72.8 mm, vias 4 -> 2
- net GPIO2_12VOut: track 79.2 -> 61.8 mm, vias 2 -> 0
- net GPIO3_In: track 60.4 -> 77.6 mm, vias 3 -> 2
- net GPIO2_In: track 80.6 -> 64.4 mm, vias 2 -> 0
- net GPIO5_12VOut: track 54.0 -> 37.9 mm, vias 4 -> 1
- net GPIO3_12VOut: track 53.4 -> 68.9 mm
- net +12V: track 110.9 -> 125.6 mm, vias 6 -> 3
- net GPIO1_12VOut: track 45.9 -> 59.3 mm
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- added copper zone on In1.Cu, net +3.3V
- added copper zone on F.Cu, net GND
- added copper zone on In2.Cu, net GND
- removed copper zone on In2.Cu, net +3.3V
- removed copper zone on In1.Cu, net GND

Commit message: few small changes
Changed lines of the file:
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@@
       (drillshape 0)
       (scaleselection 1)
-      (outputdirectory "")
+      (outputdirectory "Gerber/")
     )
   )
@@
     (fp_line (start 1 0.6) (end -0.7 0.6)
       (stroke (width 0.1) (type solid)) (layer "B.Fab"))
-    (pad "1" smd roundrect (at -1.025 0 180) (size 1.15 1.4) (layers "B.Cu" "B.Paste" "B.Mask") (roundrect_rratio 0.217391)
+    (pad "1" smd roundrect (at -1.025 0 180) (size 1.15 1.4) (layers "B.Cu" "B.Paste" "B.Mask") (roundrect_rratio 0.2173913043)
       (net 1 "GND") (pinfunction "K") (pintype "passive"))
-    (pad "2" smd roundrect (at 1.025 0 180) (size 1.15 1.4) (layers "B.Cu" "B.Paste" "B.Mask") (roundrect_rratio 0.217391)
+    (pad "2" smd roundrect (at 1.025 0 180) (size 1.15 1.4) (layers "B.Cu" "B.Paste" "B.Mask") (roundrect_rratio 0.2173913043)
       (net 14 "Net-(12VGood1-A)") (pinfunction "A") (pintype "passive"))
     (model "${KICAD6_3DMODEL_DIR}/LED_SMD.3dshapes/LED_0805_2012Metric.wrl"
@@
     (fp_line (start 1 0.625) (end 1 -0.625)
       (stroke (width 0.1) (type solid)) (layer "B.Fab"))
-    (pad "1" smd roundrect (at -1.0375 0 180) (size 1.175 1.45) (layers "B.Cu" "B.Paste" "B.Mask") (roundrect_rratio 0.212766)
+    (pad "1" smd roundrect (at -1.0375 0 180) (size 1.175 1.45) (layers "B.Cu" "B.Paste" "B.Mask") (roundrect_rratio 0.2127659574)
       (net 25 "+12V") (pintype "passive"))
-    (pad "2" smd roundrect (at 1.0375 0 180) (size 1.175 1.45) (layers "B.Cu" "B.Paste" "B.Mask") (roundrect_rratio 0.212766)
+    (pad "2" smd roundrect (at 1.0375 0 180) (size 1.175 1.45) (layers "B.Cu" "B.Paste" "B.Mask") (roundrect_rratio 0.2127659574)
       (net 1 "GND") (pintype "passive"))
     (model "${KICAD6_3DMODEL_DIR}/Capacitor_SMD.3dshapes/C_0805_2012Metric.wrl"
@@
     (fp_line (start 1 0.625) (end 1 -0.625)
       (stroke (width 0.1) (type solid)) (layer "B.Fab"))
-    (pad "1" smd roundrect (at -1.0375 0 180) (size 1.175 1.45) (layers "B.Cu" "B.Paste" "B.Mask") (roundrect_rratio 0.212766)
+    (pad "1" smd roundrect (at -1.0375 0 180) (size 1.175 1.45) (layers "B.Cu" "B.Paste" "B.Mask") (roundrect_rratio 0.2127659574)
       (net 7 "+BATT") (pintype "passive"))
-    (pad "2" smd roundrect (at 1.0375 0 180) (size 1.175 1.45) (layers "B.Cu" "B.Paste" "B.Mask") (roundrect_rratio 0.212766)
+    (pad "2" smd roundrect (at 1.0375 0 180) (size 1.175 1.45) (layers "B.Cu" "B.Paste" "B.Mask") (roundrect_rratio 0.2127659574)
       (net 1 "GND") (pintype "passive"))
     (model "${KICAD6_3DMODEL_DIR}/Capacitor_SMD.3dshapes/C_0805_2012Metric.wrl"
@@
     (fp_line (start 4.11 2.7) (end 4.11 -2.7)
       (stroke (width 0.1) (type solid)) (layer "B.Fab"))
-    (pad "1" smd roundrect (at -5.04 2.28 90) (size 2.2 1.2) (layers "B.Cu" "B.Paste" "B.Mask") (roundrect_rratio 0.208333)
+    (pad "1" smd roundrect (at -5.04 2.28 90) (size 2.2 1.2) (layers "B.Cu" "B.Paste" "B.Mask") (roundrect_rratio 0.2083333333)
       (net 59 "Net-(JP1-B)") (pinfunction "GND") (pintype "power_in"))
-    (pad "2" smd roundrect (at -0.415 -1.525 90) (size 3.05 2.75) (layers "B.Cu" "B.Paste") (roundrect_rratio 0.090909)
+    (pad "2" smd roundrect (at -0.415 -1.525 90) (size 3.05 2.75) (layers "B.Cu" "B.Paste") (roundrect_rratio 0.09090909091)
       (net 25 "+12V") (pinfunction "VO") (pintype "power_out"))
-    (pad "2" smd roundrect (at -0.415 1.525 90) (size 3.05 2.75) (layers "B.Cu" "B.Paste") (roundrect_rratio 0.090909)
+    (pad "2" smd roundrect (at -0.415 1.525 90) (size 3.05 2.75) (layers "B.Cu" "B.Paste") (roundrect_rratio 0.09090909091)
       (net 25 "+12V") (pinfunction "VO") (pintype "power_out"))
-    (pad "2" smd roundrect (at 1.26 0 90) (size 6.4 5.8) (layers "B.Cu" "B.Mask") (roundrect_rratio 0.043103)
+    (pad "2" smd roundrect (at 1.26 0 90) (size 6.4 5.8) (layers "B.Cu" "B.Mask") (roundrect_rratio 0.04310293103)
       (net 25 "+12V") (pinfunction "VO") (pintype "power_out"))
-    (pad "2" smd roundrect (at 2.935 -1.525 90) (size 3.05 2.75) (layers "B.Cu" "B.Paste") (roundrect_rratio 0.090909)
+    (pad "2" smd roundrect (at 2.935 -1.525 90) (size 3.05 2.75) (layers "B.Cu" "B.Paste") (roundrect_rratio 0.09090909091)
       (net 25 "+12V") (pinfunction "VO") (pintype "power_out"))
-    (pad "2" smd roundrect (at 2.935 1.525 90) (size 3.05 2.75) (layers "B.Cu" "B.Paste") (roundrect_rratio 0.090909)
+    (pad "2" smd roundrect (at 2.935 1.525 90) (size 3.05 2.75) (layers "B.Cu" "B.Paste") (roundrect_rratio 0.09090909091)
       (net 25 "+12V") (pinfunction "VO") (pintype "power_out"))
-    (pad "3" smd roundrect (at -5.04 -2.28 90) (size 2.2 1.2) (layers "B.Cu" "B.Paste" "B.Mask") (roundrect_rratio 0.208333)
+    (pad "3" smd roundrect (at -5.04 -2.28 90) (size 2.2 1.2) (layers "B.Cu" "B.Paste" "B.Mask") (roundrect_rratio 0.2083333333)
       (net 7 "+BATT") (pinfunction "VI") (pintype "power_in"))
     (model "${KICAD6_3DMODEL_DIR}/Package_TO_SOT_SMD.3dshapes/TO-252-2.wrl"
@@
     (fp_line (start 1 0.625) (end 1 -0.625)
       (stroke (width 0.1) (type solid)) (layer "B.Fab"))
-    (pad "1" smd roundrect (at -1.0375 0 270) (size 1.175 1.45) (layers "B.Cu" "B.Paste" "B.Mask") (roundrect_rratio 0.212766)
+    (pad "1" smd roundrect (at -1.0375 0 270) (size 1.175 1.45) (layers "B.Cu" "B.Paste" "B.Mask") (roundrect_rratio 0.2127659574)
       (net 8 "+5V") (pintype "passive"))
-    (pad "2" smd roundrect (at 1.0375 0 270) (size 1.175 1.45) (layers "B.Cu" "B.Paste" "B.Mask") (roundrect_rratio 0.212766)
+    (pad "2" smd roundrect (at 1.0375 0 270) (size 1.175 1.45) (layers "B.Cu" "B.Paste" "B.Mask") (roundrect_rratio 0.2127659574)
       (net 1 "GND") (pintype "passive"))
     (model "${KICAD6_3DMODEL_DIR}/Capacitor_SMD.3dshapes/C_0805_2012Metric.wrl"
@@
     (fp_line (start 1 0.625) (end 1 -0.625)
       (stroke (width 0.1) (type solid)) (layer "B.Fab"))
-    (pad "1" smd roundrect (at -1.0375 0 270) (size 1.175 1.45) (layers "B.Cu" "B.Paste" "B.Mask") (roundrect_rratio 0.212766)
+    (pad "1" smd roundrect (at -1.0375 0 270) (size 1.175 1.45) (layers "B.Cu" "B.Paste" "B.Mask") (roundrect_rratio 0.2127659574)
       (net 1 "GND") (pintype "passive"))
-    (pad "2" smd roundrect (at 1.0375 0 270) (size 1.175 1.45) (layers "B.Cu" "B.Paste" "B.Mask") (roundrect_rratio 0.212766)
+    (pad "2" smd roundrect (at 1.0375 0 270) (size 1.175 1.45) (layers "B.Cu" "B.Paste" "B.Mask") (roundrect_rratio 0.2127659574)
       (net 8 "+5V") (pintype "passive"))
     (model "${KICAD6_3DMODEL_DIR}/Capacitor_SMD.3dshapes/C_0805_2012Metric.wrl"

Commit message: production ready
Parts:
- added R48: 20R 0603, Resistor_SMD:R_0603_1608Metric_Pad0.98x0.95mm_HandSolder, B.Cu at (28.8, 30.2)
- added R50: 10kR 0603, Resistor_SMD:R_0603_1608Metric_Pad0.98x0.95mm_HandSolder, B.Cu at (33.8, 21.0)
- added R52: 10kR 0603, Resistor_SMD:R_0603_1608Metric_Pad0.98x0.95mm_HandSolder, B.Cu at (40.0, 17.2)
- added R55: 10kR 0603, Resistor_SMD:R_0603_1608Metric_Pad0.98x0.95mm_HandSolder, B.Cu at (37.0, 19.8)
- added R56: 20R 0603, Resistor_SMD:R_0603_1608Metric_Pad0.98x0.95mm_HandSolder, B.Cu at (37.5, 25.2)
- added R57: 10kR 0603, Resistor_SMD:R_0603_1608Metric_Pad0.98x0.95mm_HandSolder, B.Cu at (56.0, 30.0)
- added R58: 10kR 0603, Resistor_SMD:R_0603_1608Metric_Pad0.98x0.95mm_HandSolder, B.Cu at (50.5, 29.5)
- added R59: 10kR 0603, Resistor_SMD:R_0603_1608Metric_Pad0.98x0.95mm_HandSolder, B.Cu at (62.2, 18.0)
- added R60: 10kR 0603, Resistor_SMD:R_0603_1608Metric_Pad0.98x0.95mm_HandSolder, B.Cu at (55.0, 44.5)
- moved C6 0.77 mm to (39.9, 24.3)
- moved C8 0.77 mm to (39.9, 26.0)
- renumbered 12VGood to 12VGood1, 3V3Good to 3V3Good1, 5VGood to 5VGood1, Error to Error1, Heart to Heart1
Connections:
- U3 pad 11: /SPI2_MOSI_RGBLED -> Net-(U3-PC3)
- U3 pad 29: /SPI2_SCK_RGBLED -> Net-(U3-PB10)
Routing:
- net +3.3V: track 63.7 -> 89.5 mm, vias 13 -> 15
- net /SPI2_MOSI_RGBLED: track 43.4 -> 49.8 mm, vias 2 -> 4
- net /SPI2_SCK_RGBLED: track 29.4 -> 24.3 mm
- net /nCS_Display: track 23.5 -> 27.9 mm, vias 1 -> 2
- net GND: track 146.2 -> 149.5 mm, vias 73 -> 74
- net Net-(U3-PC3): track 0.00 -> 3.06 mm
- net Net-(U3-PB10): track 0.00 -> 2.81 mm
- net ADC2_CTRL: track 35.1 -> 37.6 mm, vias 2 -> 3
- net Reset: track 82.8 -> 81.0 mm
- net ADC0_CTRL: track 41.2 -> 43.0 mm
- net /D_nC_Display: track 19.8 -> 21.1 mm, vias 1 -> 2
- net /SPI1_MOSI_Display: track 18.5 -> 17.6 mm, vias 2 -> 0
- net GPIO4_In: track 38.1 -> 37.3 mm
- net GPIO5_In: track 40.5 -> 39.9 mm
- net /SPI1_SCK_Display: track 22.2 -> 21.7 mm, vias 4 -> 2
