File: ECAD/ConnectorIntefaceBoard/ConnectorInterfaceBoard/ConnectorInterfaceBoard.kicad_pcb (KiCad board)
At the start: 2 copper layers, 4 parts, among them J1 Conn_01x07, J2 Conn_01x06, J3 Conn_01x05, J4 WE 62702621621

Commit message: few small changes
Other:
- board outline added: 56.9 x 16.8 mm
Changed lines of the file:
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@@
     (pad_to_mask_clearance 0)
     (pcbplotparams
-      (layerselection 0x00010fc_ffffffff)
+      (layerselection 0x00010f0_ffffffff)
       (plot_on_all_layers_selection 0x0000000_00000000)
       (disableapertmacros false)
@@
       (outputformat 1)
       (mirror false)
-      (drillshape 1)
+      (drillshape 0)
       (scaleselection 1)
       (outputdirectory "")
@@
         (effects (font (size 1 1) (thickness 0.15)))
     )
+    (fp_text user "." (at -6 -3.4 unlocked) (layer "F.SilkS")
+        (effects (font (size 1 1) (thickness 0.1)) (justify left bottom))
+    )
+    (fp_text user "5" (at 4 1.2 unlocked) (layer "F.SilkS")
+        (effects (font (size 1 1) (thickness 0.1)) (justify left bottom))
+    )
+    (fp_text user "4" (at 2.6 4 unlocked) (layer "F.SilkS")
+        (effects (font (size 1 1) (thickness 0.1)) (justify left bottom))
+    )
+    (fp_text user "1" (at -4.2 -2 unlocked) (layer "F.SilkS")
+        (effects (font (size 1 1) (thickness 0.1)) (justify left bottom))
+    )
     (fp_text user "3" (at -3.6 4 unlocked) (layer "F.SilkS")
         (effects (font (size 1 1) (thickness 0.1)) (justify left bottom))
     )
-    (fp_text user "1" (at -4.2 -2 unlocked) (layer "F.SilkS")
-        (effects (font (size 1 1) (thickness 0.1)) (justify left bottom))
-    )
-    (fp_text user "." (at -6 -3.4 unlocked) (layer "F.SilkS")
-        (effects (font (size 1 1) (thickness 0.1)) (justify left bottom))
-    )
-    (fp_text user "5" (at 4 1.2 unlocked) (layer "F.SilkS")
-        (effects (font (size 1 1) (thickness 0.1)) (justify left bottom))
-    )
     (fp_text user "2" (at -4.8 1.2 unlocked) (layer "F.SilkS")
         (effects (font (size 1 1) (thickness 0.1)) (justify left bottom))
     )
+    (fp_text user "1" (at -0.6 -1.8 unlocked) (layer "F.SilkS")
+        (effects (font (size 1 1) (thickness 0.1)) (justify left bottom))
+    )
     (fp_text user "6" (at 3.8 -1.6 unlocked) (layer "F.SilkS")
-        (effects (font (size 1 1) (thickness 0.1)) (justify left bottom))
-    )
-    (fp_text user "4" (at 2.6 4 unlocked) (layer "F.SilkS")
-        (effects (font (size 1 1) (thickness 0.1)) (justify left bottom))
-    )
-    (fp_text user "1" (at -0.6 -1.8 unlocked) (layer "F.SilkS")
         (effects (font (size 1 1) (thickness 0.1)) (justify left bottom))
     )
@@
     (fp_circle (center 0 0) (end 5.9055 0)
       (stroke (width 0.1) (type default)) (fill none) (layer "F.SilkS"))
-    (pad "1" thru_hole circle (at -2.1336 -1.1938) (size 1.5 1.5) (drill 1.32) (layers "*.Cu" "*.Mask")
+    (pad "1" thru_hole circle (at -2.1336 -1.1938) (size 1.52 1.52) (drill 1.32) (layers "*.Cu" "*.Mask")
       (net 1 "GPIO1_out{slash}in") (pinfunction "Pin_1") (pintype "passive"))
-    (pad "2" thru_hole circle (at -1.9812 0.508) (size 1.5 1.5) (drill 1.32) (layers "*.Cu" "*.Mask")
+    (pad "2" thru_hole circle (at -1.9812 0.508) (size 1.52 1.52) (drill 1.32) (layers "*.Cu" "*.Mask")
       (net 2 "GPIO2_out{slash}in") (pinfunction "Pin_2") (pintype "passive"))
-    (pad "3" thru_hole circle (at -1.27 2.0828) (size 1.5 1.5) (drill 1.32) (layers "*.Cu" "*.Mask")
+    (pad "3" thru_hole circle (at -1.27 2.0828) (size 1.52 1.52) (drill 1.32) (layers "*.Cu" "*.Mask")
       (net 3 "GPIO3_out{slash}in") (pinfunction "Pin_3") (pintype "passive"))
-    (pad "4" thru_hole circle (at 1.27 2.0828) (size 1.5 1.5) (drill 1.32) (layers "*.Cu" "*.Mask")
+    (pad "4" thru_hole circle (at 1.27 2.0828) (size 1.52 1.52) (drill 1.32) (layers "*.Cu" "*.Mask")
       (net 4 "GPIO4_out{slash}in") (pinfunction "Pin_4") (pintype "passive"))
-    (pad "5" thru_hole circle (at 1.9812 0.508) (size 1.5 1.5) (drill 1.32) (layers "*.Cu" "*.Mask")
+    (pad "5" thru_hole circle (at 1.9812 0.508) (size 1.52 1.52) (drill 1.32) (layers "*.Cu" "*.Mask")
       (net 5 "GPIO5_out{slash}in") (pinfunction "Pin_5") (pintype "passive"))
-    (pad "6" thru_hole circle (at 2.1336 -1.1938) (size 1.5 1.5) (drill 1.32) (layers "*.Cu" "*.Mask")
+    (pad "6" thru_hole circle (at 2.1336 -1.1938) (size 1.52 1.52) (drill 1.32) (layers "*.Cu" "*.Mask")
       (net 6 "GPIO6_out{slash}in") (pinfunction "Pin_6") (pintype "passive"))
-    (pad "7" thru_hole circle (at 0 -0.6858) (size 1.5 1.5) (drill 1.32) (layers "*.Cu" "*.Mask")
-      (net 7 "GND") (pinfunction "Pin_7") (pintype "passive") (thermal_bridge_angle 0))
+    (pad "7" thru_hole circle (at 0 -0.6858) (size 1.52 1.52) (drill 1.32) (layers "*.Cu" "*.Mask")
+      (net 7 "GND") (pinfunction "Pin_7") (pintype "passive"))
+    (model "E:/Privat/Git/KiCADLib/Library.pretty/3D File RT3MP.STP"
+      (offset (xyz 0 0 16.5))
+      (scale (xyz 1 1 1))
+      (rotate (xyz 0 -90 0))
+    )
   )
   (footprint "Library:MiniXLR_5Pin" (layer "F.Cu")
@@
         (effects (font (size 1 1) (thickness 0.15)))
     )
+    (fp_text user "2" (at -3.8 4 unlocked) (layer "F.SilkS")
+        (effects (font (size 1 1) (thickness 0.1)) (justify left bottom))
+    )
+    (fp_text user "." (at -6.8 -2.8 unlocked) (layer "F.SilkS")
+        (effects (font (size 1 1) (thickness 0.1)) (justify left bottom))
+    )
+    (fp_text user "4" (at 3.8 -1 unlocked) (layer "F.SilkS")
+        (effects (font (size 1 1) (thickness 0.1)) (justify left bottom))
+    )
     (fp_text user "1" (at -4.4 -1.4 unlocked) (layer "F.SilkS")
         (effects (font (size 1 1) (thickness 0.1)) (justify left bottom))
     )
+    (fp_text user "5" (at -0.6 -1.6 unlocked) (layer "F.SilkS")
+        (effects (font (size 1 1) (thickness 0.1)) (justify left bottom))
+    )
     (fp_text user "3" (at 2.4 4 unlocked) (layer "F.SilkS")
-        (effects (font (size 1 1) (thickness 0.1)) (justify left bottom))
-    )
-    (fp_text user "4" (at 3.8 -1 unlocked) (layer "F.SilkS")
-        (effects (font (size 1 1) (thickness 0.1)) (justify left bottom))
-    )
-    (fp_text user "5" (at -0.6 -1.6 unlocked) (layer "F.SilkS")
-        (effects (font (size 1 1) (thickness 0.1)) (justify left bottom))
-    )
-    (fp_text user "." (at -6.8 -2.8 unlocked) (layer "F.SilkS")
-        (effects (font (size 1 1) (thickness 0.1)) (justify left bottom))
-    )
-    (fp_text user "2" (at -3.8 4 unlocked) (layer "F.SilkS")
         (effects (font (size 1 1) (thickness 0.1)) (justify left bottom))
     )
@@
       (net 14 "CAN1_P") (pinfunction "Pin_4") (pintype "passive"))
     (pad "5" thru_hole circle (at 0 0) (size 2 2) (drill 1.6) (layers "*.Cu" "*.Mask")
-      (net 7 "GND") (pinfunction "Pin_5") (pintype "passive") (thermal_bridge_angle 0))
+      (net 7 "GND") (pinfunction "Pin_5") (pintype "passive"))
+    (model "E:/Privat/Git/KiCADLib/Library.pretty/3D File RT3MP.STP"
+      (offset (xyz 0 0 16.5))
+      (scale (xyz 1 1 1))
+      (rotate (xyz 0 -90 90))
+    )
   )
   (footprint "Library:MiniXLR_6Pin" (layer "F.Cu")
@@
         (effects (font (size 1 1) (thickness 0.1)) (justify left bottom))
     )
+    (fp_text user "6" (at -0.6 -1.4 unlocked) (layer "F.SilkS")
+        (effects (font (size 1 1) (thickness 0.1)) (justify left bottom))
+    )
+    (fp_text user "4" (at 3.8 2.2 unlocked) (layer "F.SilkS")
+        (effects (font (size 1 1) (thickness 0.1)) (justify left bottom))
+    )
+    (fp_text user "2" (at -4.8 2.2 unlocked) (layer "F.SilkS")
+        (effects (font (size 1 1) (thickness 0.1)) (justify left bottom))
+    )
+    (fp_text user "5" (at 3.2 -2.2 unlocked) (layer "F.SilkS")
+        (effects (font (size 1 1) (thickness 0.1)) (justify left bottom))
+    )
+    (fp_text user "1" (at -4.2 -2.2 unlocked) (layer "F.SilkS")
+        (effects (font (size 1 1) (thickness 0.1)) (justify left bottom))
+    )
     (fp_text user "." (at -6 -3.8 unlocked) (layer "F.SilkS")
-        (effects (font (size 1 1) (thickness 0.1)) (justify left bottom))
-    )
-    (fp_text user "4" (at 3.8 2.2 unlocked) (layer "F.SilkS")
-        (effects (font (size 1 1) (thickness 0.1)) (justify left bottom))
-    )
-    (fp_text user "1" (at -4.2 -2.2 unlocked) (layer "F.SilkS")
-        (effects (font (size 1 1) (thickness 0.1)) (justify left bottom))
-    )
-    (fp_text user "5" (at 3.2 -2.2 unlocked) (layer "F.SilkS")
-        (effects (font (size 1 1) (thickness 0.1)) (justify left bottom))
-    )
-    (fp_text user "6" (at -0.6 -1.4 unlocked) (layer "F.SilkS")
-        (effects (font (size 1 1) (thickness 0.1)) (justify left bottom))
-    )
-    (fp_text user "2" (at -4.8 2.2 unlocked) (layer "F.SilkS")
         (effects (font (size 1 1) (thickness 0.1)) (justify left bottom))
     )
@@
       (net 12 "Analog3_In") (pinfunction "Pin_5") (pintype "passive"))
     (pad "6" thru_hole circle (at 0 0) (size 2 2) (drill 1.6) (layers "*.Cu" "*.Mask")
-      (net 7 "GND") (pinfunction "Pin_6") (pintype "passive") (thermal_bridge_angle 0))
-  )
-  (gr_rect (start 14.6882 28.67) (end 19.8882 11.97)
+      (net 7 "GND") (pinfunction "Pin_6") (pintype "passive"))
+    (model "E:/Privat/Git/KiCADLib/Library.pretty/3D File RT3MP.STP"
+      (offset (xyz 0 0 16.5))
+      (scale (xyz 1 1 1))
+      (rotate (xyz 0 -90 0))
+    )
+  )
+  (gr_rect (start 14.6882 11.97) (end 19.8882 28.67)
     (stroke (width 0.1) (type default)) (fill none) (layer "B.SilkS"))
   (gr_rect (start 11.938 11.938) (end 68.834 28.702)
-    (stroke (width 0.15) (type default)) (fill none) (layer "Margin"))
+    (stroke (width 0.15) (type default)) (fill none) (layer "Edge.Cuts"))
   (gr_circle (center 45.847 20.4978) (end 54.247 20.4978)
     (stroke (width 0.2) (type default)) (fill none) (layer "B.Fab"))

Commit message: production ready
Routing:
- net GND: track 2.51 -> 11.8 mm, vias 6 -> 23
Changed lines of the file:
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@@
       (drillshape 0)
       (scaleselection 1)
-      (outputdirectory "")
+      (outputdirectory "Gerber")
     )
   )
@@
   (segment (start 14.332046 26.813404) (end 15.2908 25.85465) (width 0.75) (layer "B.Cu") (net 6))
   (segment (start 16.4338 22.225) (end 16.7132 22.225) (width 0.75) (layer "B.Cu") (net 6))
+  (segment (start 62.865 18.885) (end 64 17.75) (width 0.75) (layer "F.Cu") (net 7))
+  (segment (start 62.865 20.3708) (end 62.865 18.885) (width 0.75) (layer "F.Cu") (net 7))
+  (segment (start 28.829 18.921) (end 30 17.75) (width 0.75) (layer "F.Cu") (net 7))
+  (segment (start 28.829 19.685) (end 28.829 18.921) (width 0.75) (layer "F.Cu") (net 7))
+  (via (at 58 19.25) (size 0.8) (drill 0.4) (layers "F.Cu" "B.Cu") (free) (net 7))
   (via (at 20.828 24.4856) (size 0.8) (drill 0.4) (layers "F.Cu" "B.Cu") (free) (net 7))
+  (via (at 26.25 17) (size 0.8) (drill 0.4) (layers "F.Cu" "B.Cu") (free) (net 7))
+  (via (at 21 22.2116) (size 0.8) (drill 0.4) (layers "F.Cu" "B.Cu") (free) (net 7))
   (via (at 22.9108 25.7556) (size 0.8) (drill 0.4) (layers "F.Cu" "B.Cu") (free) (net 7))
+  (via (at 30 17.75) (size 0.8) (drill 0.4) (layers "F.Cu" "B.Cu") (net 7))
   (via (at 14.5796 18.3896) (size 0.8) (drill 0.4) (layers "F.Cu" "B.Cu") (free) (net 7))
+  (via (at 57.5 24.75) (size 0.8) (drill 0.4) (layers "F.Cu" "B.Cu") (free) (net 7))
   (via (at 24.5872 24.9936) (size 0.8) (drill 0.4) (layers "F.Cu" "B.Cu") (free) (net 7))
+  (via (at 35.25 17.25) (size 0.8) (drill 0.4) (layers "F.Cu" "B.Cu") (free) (net 7))
+  (via (at 13.5 19.75) (size 0.8) (drill 0.4) (layers "F.Cu" "B.Cu") (free) (net 7))
+  (via (at 46.25 17) (size 0.8) (drill 0.4) (layers "F.Cu" "B.Cu") (free) (net 7))
   (via (at 28.8036 25.7556) (size 0.8) (drill 0.4) (layers "F.Cu" "B.Cu") (free) (net 7))
+  (via (at 51.5 24.75) (size 0.8) (drill 0.4) (layers "F.Cu" "B.Cu") (free) (net 7))
+  (via (at 38.75 22) (size 0.8) (drill 0.4) (layers "F.Cu" "B.Cu") (free) (net 7))
+  (via (at 52.5 17.75) (size 0.8) (drill 0.4) (layers "F.Cu" "B.Cu") (free) (net 7))
   (via (at 31.3436 25.8064) (size 0.8) (drill 0.4) (layers "F.Cu" "B.Cu") (free) (net 7))
+  (via (at 44.25 17.25) (size 0.8) (drill 0.4) (layers "F.Cu" "B.Cu") (net 7))
+  (via (at 13.25 16.75) (size 0.8) (drill 0.4) (layers "F.Cu" "B.Cu") (free) (net 7))
+  (via (at 39 18.25) (size 0.8) (drill 0.4) (layers "F.Cu" "B.Cu") (free) (net 7))
+  (via (at 64 17.75) (size 0.8) (drill 0.4) (layers "F.Cu" "B.Cu") (net 7))
+  (via (at 60.75 16.5) (size 0.8) (drill 0.4) (layers "F.Cu" "B.Cu") (free) (net 7))
+  (via (at 22 19.75) (size 0.8) (drill 0.4) (layers "F.Cu" "B.Cu") (free) (net 7))
+  (segment (start 45.8216 20.3962) (end 45.8216 18.8216) (width 0.75) (layer "B.Cu") (net 7))
+  (segment (start 45.8216 18.8216) (end 44.25 17.25) (width 0.75) (layer "B.Cu") (net 7))
   (segment (start 62.865 20.3708) (end 62.865 20.9042) (width 0.75) (layer "B.Cu") (net 7))
   (segment (start 62.865 20.9042) (end 61.468 22.3012) (width 0.75) (layer "B.Cu") (net 7))
@@
   (segment (start 23.814451 23.785148) (end 23.814451 25.559112) (width 0.3) (layer "F.Cu") (net 14))
   (segment (start 25.317939 27.0626) (end 34.29037 27.0626) (width 0.3) (layer "F.Cu") (net 14))
+  (segment (start 19.858628 23.25) (end 19.570228 22.9616) (width 0.3) (layer "F.Cu") (net 14))
   (segment (start 34.29037 27.0626) (end 34.54037 26.8126) (width 0.3) (layer "F.Cu") (net 14))
+  (segment (start 21.486228 23.236228) (end 21.472456 23.25) (width 0.3) (layer "F.Cu") (net 14))
+  (segment (start 19.570228 22.9616) (end 18.5166 22.9616) (width 0.3) (layer "F.Cu") (net 14))
   (segment (start 18.5166 22.9616) (end 17.9832 23.495) (width 0.3) (layer "F.Cu") (net 14))
-  (segment (start 21.760856 22.9616) (end 18.5166 22.9616) (width 0.3) (layer "F.Cu") (net 14))
+  (segment (start 21.472456 23.25) (end 19.858628 23.25) (width 0.3) (layer "F.Cu") (net 14))
   (segment (start 23.814451 25.559112) (end 25.317939 27.0626) (width 0.3) (layer "F.Cu") (net 14))
-  (segment (start 21.862545 22.859911) (end 21.760856 22.9616) (width 0.3) (layer "F.Cu") (net 14))
   (via (at 34.54037 26.8126) (size 0.8) (drill 0.4) (layers "F.Cu" "B.Cu") (net 14))
   (via (at 23.814451 23.785148) (size 0.8) (drill 0.4) (layers "F.Cu" "B.Cu") (net 14))
-  (via (at 21.862545 22.859911) (size 0.8) (drill 0.4) (layers "F.Cu" "B.Cu") (net 14))
+  (via (at 21.486228 23.236228) (size 0.8) (drill 0.4) (layers "F.Cu" "B.Cu") (net 14))
+  (segment (start 21.486228 23.236228) (end 21.628809 23.236228) (width 0.3) (layer "B.Cu") (net 14))
   (segment (start 35.36297 27.6352) (end 63.9064 27.6352) (width 0.3) (layer "B.Cu") (net 14))
   (segment (start 34.54037 26.8126) (end 35.36297 27.6352) (width 0.3) (layer "B.Cu") (net 14))
-  (segment (start 21.862545 23.469964) (end 22.177729 23.785148) (width 0.3) (layer "B.Cu") (net 14))
   (segment (start 66.0748 25.4668) (end 66.0748 20.685) (width 0.3) (layer "B.Cu") (net 14))
   (segment (start 63.9064 27.6352) (end 66.0748 25.4668) (width 0.3) (layer "B.Cu") (net 14))
   (segment (start 66.0748 20.685) (end 65.0748 19.685) (width 0.3) (layer "B.Cu") (net 14))
+  (segment (start 21.628809 23.236228) (end 22.177729 23.785148) (width 0.3) (layer "B.Cu") (net 14))
   (segment (start 22.177729 23.785148) (end 23.814451 23.785148) (width 0.3) (layer "B.Cu") (net 14))
-  (segment (start 21.862545 22.859911) (end 21.862545 23.469964) (width 0.3) (layer "B.Cu") (net 14))
   (zone (net 7) (net_name "GND") (layer "F.Cu") (hatch edge 0.5)
     (connect_pads (clearance 0.5))
